File: modules/HID module/board/board.kicad_pcb (KiCad board)
At the start: 2 copper layers, 45 x 30 mm, 30 parts, among them J1 USB_C_Receptacle_USB2.0, J2 Conn_01x06, J3 Conn_01x06, J6 Conn_01x06, SW1 RESET, U1 ESP32-WROOM-32, U2 HT7533-1-SOT89, U3 HT42B564

Commit message: PCB: USB C receptacle moved close to PCB edge
Parts:
- J1: footprint Connector_USB:USB_C_Receptacle_HRO_TYPE-C-31-M-12 -> Board:USB_C_Receptacle_HRO_TYPE-C-31-M-12
- moved J1 0.42 mm to (161.2, 90.5)
Routing:
- net GND: track 164.2 -> 153.1 mm, vias 4 -> 6
- net /DI+: track 9.42 -> 11.2 mm
- net Net-(J1-PadA5): track 13.0 -> 14.4 mm
